File: connectors.kicad_sch (KiCad schematic)
At the start: 9 parts, among them J13 SM08B-SRSS-TB_LF__SN_, J14 Conn_01x01, J15 Conn_01x01

Commit message: affected footprints
Parts:
- added TP1, TP10, TP11, TP12, TP8, TP9: TestPoint, TestPoint:TestPoint_Loop_D1.80mm_Drill1.0mm_Beaded, symbol Connector:TestPoint
- J14, J15: footprint (none) -> TestPoint:TestPoint_Pad_2.0x2.0mm; now left out of the parts list
- TP2, TP3, TP4, TP5, TP6, TP7: footprint (none) -> TestPoint:TestPoint_Loop_D1.80mm_Drill1.0mm_Beaded; now left out of the parts list
Connections:
- net SWCLK renamed SWCLK1
- net SWDIO renamed SWDIO1
- new net SWCLK2: TP1.1
- new net SWCLK3: TP9.1
- new net SWCLK4: TP11.1
- new net SWDIO2: TP8.1
- new net SWDIO3: TP10.1
- new net SWDIO4: TP12.1

Commit message: minor fixes
Parts:
- removed TP4, TP5, TP6, TP7: TestPoint, TestPoint:TestPoint_Loop_D1.80mm_Drill1.0mm_Beaded, symbol Connector:TestPoint
- J14, J15: footprint TestPoint:TestPoint_Pad_2.0x2.0mm -> TestPoint:TestPoint_Pad_4.0x4.0mm
